File: bluePillG.sch (KiCad schematic (older format))
At the start: 34 parts, among them IC1 STM32G431C6T6, J1 Conn_02x03_Odd_Even, J2 Conn_01x20_Male, J3 Conn_01x04_Male, J4 Conn_01x20_Male, U1 LM1117-3.3, Y1 32.768kHz, Y2 8MHz

Commit message: board
Parts:
- IC1: symbol STM32G431C6T6:STM32G431C6T6 -> bluePillG-rescue:STM32G431C6T6-STM32G431C6T6
- S1: symbol FSM4JH:FSM4JH -> bluePillG-rescue:FSM4JH-FSM4JH
- U1: footprint digikey-footprints:SOT-223-4 -> mod:SOT-223-4
Connections:
- net +3.3V is gone; now on net +3V3: C14.1, J3.1 (Pin_1)
Changed lines of the file:
@@
 $EndDescr
 $Comp
-L STM32G431C6T6:STM32G431C6T6 IC1
+L bluePillG-rescue:STM32G431C6T6-STM32G431C6T6 IC1
 U 1 1 60339AE3
 P 5050 3200
@@
 $EndComp
 $Comp
-L FSM4JH:FSM4JH S1
+L bluePillG-rescue:FSM4JH-FSM4JH S1
 U 1 1 6035339B
 P 1050 3100
@@
 F 0 "U1" H 1450 5192 50  0000 C CNN
 F 1 "LM1117-3.3" H 1450 5101 50  0000 C CNN
-F 2 "digikey-footprints:SOT-223-4" H 1450 4950 50  0001 C CNN
+F 2 "mod:SOT-223-4" H 1450 4950 50  0001 C CNN
 F 3 "http://www.ti.com/lit/ds/symlink/lm1117.pdf" H 1450 4950 50  0001 C CNN
 	1    1450 4950
@@
 Wire Wire Line
 	1750 6450 2000 6450
+$Comp
+L power:+3.3V #PWR?
+U 1 1 6037AECF
+P 8150 1800
+F 0 "#PWR?" H 8150 1650 50  0001 C CNN
+F 1 "+3.3V" H 8165 1973 50  0000 C CNN
+F 2 "" H 8150 1800 50  0001 C CNN
+F 3 "" H 8150 1800 50  0001 C CNN
+	1    8150 1800
+	1    0    0    -1
+$EndComp
 $EndSCHEMATC
