File: bluePillG.kicad_pcb (KiCad board)
At the start: 2 copper layers, 35.6 x 50.8 mm, 34 parts, among them IC1 STM32G431C6T6, J1 Conn_02x03_Odd_Even, J2 Conn_01x20_Male, J3 Conn_01x04_Male, J4 Conn_01x20_Male, U1 LM1117-3.3, Y1 32.768kHz, Y2 8MHz

Commit message: schematics
Other:
- board text added: "+3V3"
- board text added: "+5V"
- board text added: "BOOT0"
- board text added: "GND"
- board text added: "PA0"
- board text added: "PA1"
- board text added: "PA10"
- board text added: "PA11"
- board text added: "PA12"
- board text added: "PA15"
- board text added: "PA2"
- board text added: "PA3"
- board text added: "PA4"
- board text added: "PA5"
- board text added: "PA6"
- board text added: "PA7"
- board text added: "PA8"
- board text added: "PA9"
- board text added: "PB0"
- board text added: "PB1"
- board text added: "PB10"
- board text added: "PB11"
- board text added: "PB12"
- board text added: "PB13"
- board text added: "PB14"
- board text added: "PB15"
- board text added: "PB2"
- board text added: "PB3"
- board text added: "PB4"
- board text added: "PB5"
- board text added: "PB6"
- board text added: "PB7"
- board text added: "PB9"
- board text added: "PC13"
- board text added: "RST"

Commit message: blinker example
Parts:
- J2, J4: moved to B.Cu
- turned J2 to 180 degrees
- turned J4 to 180 degrees
