File: board-v2/mcu.sch (KiCad schematic (older format))
At the start: 36 parts

Commit message: board v2
Parts:
- added D3: LED, LED_SMD:LED_0805_2012Metric, symbol Device:LED
- added H1, H2, H3, H4: MountingHole_Pad, MountingHole:MountingHole_3.2mm_M3_Pad_Via, symbol Mechanical:MountingHole_Pad
- added J10, J9: Conn_02x02_Top_Bottom, Connector_PinSocket_2.54mm:PinSocket_2x02_P2.54mm_Vertical, symbol Connector_Generic:Conn_02x02_Top_Bottom
- added J4, J5: Conn_01x02_Male, Connector_PinSocket_2.54mm:PinSocket_1x02_P2.54mm_Vertical, symbol Connector:Conn_01x02_Male
- added J6, J7, J8: Conn_01x10_Male, Connector_PinSocket_2.54mm:PinSocket_1x10_P2.54mm_Vertical, symbol Connector:Conn_01x10_Male
- added R5: 2.2k, Resistor_SMD:R_0603_1608Metric, symbol Device:R
- C1, C10, C11, C12, C13, C14, C15, C16, C17, C18, C19, C2, C3, C4, C5, C6, C7, C8, C9: renamed from C?; footprint (none) -> Capacitor_SMD:C_0603_1608Metric
- D1: renamed from D?; footprint Diode_THT:D_DO-41_SOD81_P10.16mm_Horizontal -> Diode_SMD:D_SOD-123
- D2: renamed from D?; footprint (none) -> LED_SMD:LED_0805_2012Metric
- F1: renamed from F?; footprint (none) -> Resistors:1206
- FB1, FB2: renamed from FB?; footprint (none) -> Resistors:0603
- IC1: renamed from IC?; footprint QFP50P900X900X160-48N -> STM32G431C6T6:QFP50P900X900X160-48N
- J1: renamed from J?; footprint (none) -> Connector_PinSocket_2.54mm:PinSocket_2x05_P2.54mm_Vertical
- J2, J3: renamed from J?; footprint (none) -> Connector_PinSocket_2.54mm:PinSocket_1x03_P2.54mm_Vertical
- R1, R2, R3, R4: renamed from R?; footprint (none) -> Resistor_SMD:R_0603_1608Metric
- SW1: renamed from SW?; footprint (none) -> Button_Switch_THT:SW_PUSH_6mm_H5mm
- Y1: renamed from Y?; footprint (none) -> Clocks:CRYSTAL-PTH-2X6-CYL
- Y2: renamed from Y?; footprint (none) -> Clocks:HC49U
- gave numbers to parts that had none: 1
Connections:
- net +3.3VA: no longer J3.1 (Pin_1)
- net +3.3VP: now also J3.1 (Pin_1)
- net +3V3: now also J10.1 (Pin_1), J10.2 (Pin_2), J10.3 (Pin_3), J10.4 (Pin_4), R5.1
- net +5V: now also J5.2 (Pin_2)
- net GND: now also H2.1, H4.1, J4.2 (Pin_2), J9.1 (Pin_1), J9.2 (Pin_2), J9.3 (Pin_3), J9.4 (Pin_4)
- net VCC: now also H1.1, H3.1, J4.1 (Pin_1), J5.1 (Pin_1)
- net PA2: now reaches IC1.10 (PA2)
- net PA2: now also J6.4 (Pin_4)
- net PA3: now reaches IC1.11 (PA3)
- net PA3: now also J6.5 (Pin_5)
- net PA4: now reaches IC1.12 (PA4)
- net PA4: now also J6.6 (Pin_6)
- net PA5: now reaches IC1.13 (PA5)
- net PA5: now also J6.7 (Pin_7)
- net PA6: now reaches IC1.14 (PA6)
- net PA6: now also J6.8 (Pin_8)
- net PA7: now reaches IC1.15 (PA7)
- net PA7: now also J6.9 (Pin_9)
- net PB0: now reaches IC1.16 (PB0)
- net PB0: now also J6.10 (Pin_10)
- net PB1: now reaches IC1.17 (PB1)
- net PB1: now also J7.1 (Pin_1)
- net PB2: now reaches IC1.18 (PB2)
- net PB2: now also J7.2 (Pin_2)
- net PC13: now reaches IC1.2 (PC13)
- net PC13: now also D3.1 (K), J6.1 (Pin_1)
- net PB10: now reaches IC1.22 (PB10)
- net PB10: now also J7.3 (Pin_3)
- net PB11: now reaches IC1.25 (PB11)
- net PB11: now also J7.4 (Pin_4)
- net PB12: now reaches IC1.26 (PB12)
- net PB12: now also J7.5 (Pin_5)
- net PB13: now reaches IC1.27 (PB13)
- net PB13: now also J7.6 (Pin_6)
- net PB14: now reaches IC1.28 (PB14)
- net PB14: now also J7.7 (Pin_7)
- net PB15: now reaches IC1.29 (PB15)
- net PB15: now also J7.8 (Pin_8)
- net PA8: now reaches IC1.30 (PA8)
- net PA8: now also J7.9 (Pin_9)
- net PA9: now reaches IC1.31 (PA9)
- net PA9: now also J7.10 (Pin_10)
- net PA10: now reaches IC1.32 (PA10)
- net PA10: now also J8.1 (Pin_1)
- net PA11: now reaches IC1.33 (PA11)
- net PA11: now also J8.2 (Pin_2)
- net PA12: now reaches IC1.34 (PA12)
- net PA12: now also J8.3 (Pin_3)
- net PA15: now reaches IC1.39 (PA15)
- net PA15: now also J8.4 (Pin_4)
- net PB3: now reaches IC1.40 (PB3)
- net PB3: now also J8.5 (Pin_5)
- net PB4: now reaches IC1.41 (PB4)
- net PB4: now also J8.6 (Pin_6)
- net PB5: now reaches IC1.42 (PB5)
- net PB5: now also J8.7 (Pin_7)
- net PB6: now reaches IC1.43 (PB6)
- net PB6: now also J8.8 (Pin_8)
- net PB7: now reaches IC1.44 (PB7)
- net PB7: now also J8.9 (Pin_9)
- net PB9: now reaches IC1.46 (PB9)
- net PB9: now also J8.10 (Pin_10)
- net PA0: now reaches IC1.8 (PA0)
- net PA0: now also J6.2 (Pin_2)
- net PA1: now reaches IC1.9 (PA1)
- net PA1: now also J6.3 (Pin_3)
- new net: D3.2 (A), R5.2
Other:
- note added: "JUMPER"
- moved on the sheet: J3
